Commit message: Testing with different root link

File: mico_description/robots/standalone_arm.urdf.xacro (robot description, xacro)
@@ -14,5 +14,5 @@
 	xmlns:xacro="http://ros.org/wiki/xacro" name="mico">
 	<xacro:include filename="$(find mico_description)/urdf/mico_arm.urdf.xacro" />
-	<link name="root">
+	<link name="lift_link">
 		<visual>
 			<origin xyz="0 0 0" rpy="0 0 0" />
@@ -28,4 +28,4 @@
 		</collision>
 	</link>
-	<xacro:mico_arm parent="root" xyz="0 0 0" rpy="0 0 0" />
+	<xacro:mico_arm parent="lift_link" xyz="0 0 0" rpy="0 0 0" />
 </robot>

Commit message: renamed root to mico_root

File: mico_description/robots/standalone_arm.urdf.xacro (robot description, xacro)
@@ -14,5 +14,5 @@
 	xmlns:xacro="http://ros.org/wiki/xacro" name="mico">
 	<xacro:include filename="$(find mico_description)/urdf/mico_arm.urdf.xacro" />
-	<link name="lift_link">
+	<link name="mico_root">
 		<visual>
 			<origin xyz="0 0 0" rpy="0 0 0" />
@@ -28,4 +28,4 @@
 		</collision>
 	</link>
-	<xacro:mico_arm parent="lift_link" xyz="0 0 0" rpy="0 0 0" />
+	<xacro:mico_arm parent="mico_root" xyz="0 0 0" rpy="0 0 0" />
 </robot>
